File: IMU_WheelSpeed/IMU_WheelSpeed.kicad_pcb (KiCad board)
At the start: 2 copper layers, 56.8 x 50 mm, 23 parts, among them J1 Conn_01x04_Socket, J2 CAN_IN, J3 Conn_01x03_Socket, J4 CAN_OUT, J5 PWR_IN, J7 Conn_01x06_Socket, U1 PeripheralSOM, U4 TPS71518__SC70

Commit message: made bom
Parts:
- renumbered 12V_IN to J6, IMU_SCL to TP10, IMU_SCL to TP11, 1.8V to TP3
Other:
- board text added: "+"
Changed lines of the file:
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@@
 		)
 	)
+	(footprint "UTSVT_Power:LDO_3.3_to_1.8_2.2mmx1.3mm"
+		(layer "F.Cu")
+		(at 176.3 82.7 -90)
+		(property "Reference" "U4"
+			(at 0 -0.5 -90)
+			(unlocked yes)
+			(layer "F.SilkS")
+			(effects
+				(font
+					(size 1 1)
+					(thickness 0.1)
+				)
+			)
+		)
+		(property "Value" "TPS71518__SC70"
+			(at 0 1 -90)
+			(unlocked yes)
+			(layer "F.Fab")
+			(effects
+				(font
+					(size 1 1)
+					(thickness 0.15)
+				)
+			)
+		)
+		(property "Footprint" "UTSVT_Power:LDO_3.3_to_1.8_2.2mmx1.3mm"
+			(at 0 0 -90)
+			(unlocked yes)
+			(layer "F.Fab")
+			(hide yes)
+			(effects
+				(font
+					(size 1 1)
+					(thickness 0.15)
+				)
+			)
+		)
+		(property "Datasheet" "http://www.ti.com/lit/ds/symlink/tps715.pdf"
+			(at 0 0 -90)
+			(unlocked yes)
+			(layer "F.Fab")
+			(hide yes)
+			(effects
+				(font
+					(size 1 1)
+					(thickness 0.15)
+				)
+			)
+		)
+		(property "Description" "Low-drop Voltage Regulator, Io up to 50mA, Fixed Vo 1.8V, Ignd 3.2uA , SC70."
+			(at 0 0 -90)
+			(unlocked yes)
+			(layer "F.Fab")
+			(hide yes)
+			(effects
+				(font
+					(size 1 1)
+					(thickness 0.15)
+				)
+			)
+		)
+		(property "Mouser Link" "https://www.mouser.com/ProductDetail/Texas-Instruments/TPS71518DCKR?qs=Gse6rAGbi7%2FmSAtSseH9pg%3D%3D"
+			(at 0 0 -90)
+			(unlocked yes)
+			(layer "F.Fab")
+			(hide yes)
+			(effects
+				(font
+					(size 1 1)
+					(thickness 0.15)
+				)
+			)
+		)
+		(property ki_fp_filters "*SC?70*")
+		(sheetname "Root")
+		(sheetfile "IMU_WheelSpeed.kicad_sch")
+		(attr smd)
+		(fp_rect
+			(start -1.85 3.9)
+			(end 1.65 6.1)
+			(stroke
+				(width 0.1)
+				(type default)
+			)
+			(fill none)
+			(layer "F.SilkS")
+		)
+		(fp_text user "."
+			(at -0.6 4.6 -45)
+			(unlocked yes)
+			(layer "F.SilkS")
+			(effects
+				(font
+					(size 1 1)
+					(thickness 0.1)
+				)
+				(justify left bottom)
+			)
+		)
+		(fp_text user "${REFERENCE}"
+			(at 0 2.5 -90)
+			(unlocked yes)
+			(layer "F.Fab")
+			(effects
+				(font
+					(size 1 1)
+					(thickness 0.15)
+				)
+			)
+		)
+		(pad "1" smd roundrect
+			(at -1.2 4.3 270)
+			(size 0.95 0.4)
+			(layers "F.Cu" "F.Paste" "F.Mask")
+			(roundrect_rratio 0.25)
+			(net 11 "unconnected-(U4-NC-Pad1)")
+			(pinfunction "NC")
+			(pintype "no_connect")
+			(thermal_bridge_angle 45)
+		)
+		(pad "2" smd roundrect
+			(at -1.2 4.95 270)
+			(size 0.95 0.4)
+			(layers "F.Cu" "F.Paste" "F.Mask")
+			(roundrect_rratio 0.25)
+			(net 25 "GND")
+			(pinfunction "GND")
+			(pintype "power_in")
+			(thermal_bridge_angle 45)
+		)
+		(pad "3" smd roundrect
+			(at -1.2 5.6 270)
+			(size 0.95 0.4)
+			(layers "F.Cu" "F.Paste" "F.Mask")
+			(roundrect_rratio 0.25)
+			(net 12 "unconnected-(U4-NC-Pad3)")
+			(pinfunction "NC")
+			(pintype "no_connect")
+			(thermal_bridge_angle 45)
+		)
+		(pad "4" smd roundrect
+			(at 1 5.6 270)
+			(size 0.95 0.4)
+			(layers "F.Cu" "F.Paste" "F.Mask")
+			(roundrect_rratio 0.25)
+			(net 22 "/VDD_3.3V")
+			(pinfunction "IN")
+			(pintype "power_in")
+			(thermal_bridge_angle 45)
+		)
+		(pad "5" smd roundrect
+			(at 1 4.3 270)
+			(size 0.95 0.4)
+			(layers "F.Cu" "F.Paste" "F.Mask")
+			(roundrect_rratio 0.25)
+			(net 24 "/LDO_1.8V")
+			(pinfunction "OUT")
+			(pintype "power_out")
+			(thermal_bridge_angle 45)
+		)
+	)
 	(footprint "LED_SMD:LED_0805_2012Metric"
 		(layer "F.Cu")
@@
 		(at 173.616201 98.420901 180)
 		(tags "436500215 ")
-		(property "Reference" "12V_IN"
+		(property "Reference" "J6"
 			(at -6.133799 -0.579099 90)
 			(unlocked yes)
@@
 		)
 	)
-	(footprint "UTSVT_Power:LDO_3.3_to_1.8_2.2mmx1.3mm"
-		(layer "F.Cu")
-		(at 176.35 82.7 -90)
-		(property "Reference" "U4"
-			(at -2.5 4.85 0)
-			(unlocked yes)
-			(layer "F.SilkS")
-			(effects
-				(font
-					(size 1 1)
-					(thickness 0.1)
-				)
-			)
-		)
-		(property "Value" "TPS71518__SC70"
-			(at 0 1 -90)
-			(unlocked yes)
-			(layer "F.Fab")
-			(effects
-				(font
-					(size 1 1)
-					(thickness 0.15)
-				)
-			)
-		)
-		(property "Footprint" "UTSVT_Power:LDO_3.3_to_1.8_2.2mmx1.3mm"
-			(at 0 0 -90)
-			(unlocked yes)
-			(layer "F.Fab")
-			(hide yes)
-			(effects
-				(font
-					(size 1 1)
-					(thickness 0.15)
-				)
-			)
-		)
-		(property "Datasheet" "http://www.ti.com/lit/ds/symlink/tps715.pdf"
-			(at 0 0 -90)
-			(unlocked yes)
-			(layer "F.Fab")
-			(hide yes)
-			(effects
-				(font
-					(size 1 1)
-					(thickness 0.15)
-				)
-			)
-		)
-		(property "Description" "Low-drop Voltage Regulator, Io up to 50mA, Fixed Vo 1.8V, Ignd 3.2uA , SC70."
-			(at 0 0 -90)
-			(unlocked yes)
-			(layer "F.Fab")
-			(hide yes)
-			(effects
-				(font
-					(size 1 1)
-					(thickness 0.15)
-				)
-			)
-		)
-		(property "Mouser Link" "https://www.mouser.com/ProductDetail/Texas-Instruments/TPS71518DCKR?qs=Gse6rAGbi7%2FmSAtSseH9pg%3D%3D"
-			(at 0 0 -90)
-			(unlocked yes)
-			(layer "F.Fab")
-			(hide yes)
-			(effects
-				(font
-					(size 1 1)
-					(thickness 0.15)
-				)
-			)
-		)
-		(property ki_fp_filters "*SC?70*")
-		(sheetname "Root")
-		(sheetfile "IMU_WheelSpeed.kicad_sch")
-		(attr smd)
-		(fp_rect
-			(start -1.85 3.9)
-			(end 1.65 6.1)
-			(stroke
-				(width 0.1)
-				(type default)
-			)
-			(fill none)
-			(layer "F.SilkS")
-		)
-		(fp_text user "${REFERENCE}"
-			(at 0 2.5 -90)
-			(unlocked yes)
-			(layer "F.Fab")
-			(effects
-				(font
-					(size 1 1)
-					(thickness 0.15)
-				)
-			)
-		)
-		(pad "1" smd roundrect
-			(at -1.2 4.3 270)
-			(size 0.95 0.4)
-			(layers "F.Cu" "F.Paste" "F.Mask")
-			(roundrect_rratio 0.25)
-			(net 11 "unconnected-(U4-NC-Pad1)")
-			(pinfunction "NC")
-			(pintype "no_connect")
-			(thermal_bridge_angle 45)
-		)
-		(pad "2" smd roundrect
-			(at -1.2 4.95 270)
-			(size 0.95 0.4)
-			(layers "F.Cu" "F.Paste" "F.Mask")
-			(roundrect_rratio 0.25)
-			(net 25 "GND")
-			(pinfunction "GND")
-			(pintype "power_in")
-			(thermal_bridge_angle 45)
-		)
-		(pad "3" smd roundrect
-			(at -1.2 5.6 270)
-			(size 0.95 0.4)
-			(layers "F.Cu" "F.Paste" "F.Mask")
-			(roundrect_rratio 0.25)
-			(net 12 "unconnected-(U4-NC-Pad3)")
-			(pinfunction "NC")
-			(pintype "no_connect")
-			(thermal_bridge_angle 45)
-		)
-		(pad "4" smd roundrect
-			(at 1 5.6 270)
-			(size 0.95 0.4)
-			(layers "F.Cu" "F.Paste" "F.Mask")
-			(roundrect_rratio 0.25)
-			(net 22 "/VDD_3.3V")
-			(pinfunction "IN")
-			(pintype "power_in")
-			(thermal_bridge_angle 45)
-		)
-		(pad "5" smd roundrect
-			(at 1 4.3 270)
-			(size 0.95 0.4)
-			(layers "F.Cu" "F.Paste" "F.Mask")
-			(roundrect_rratio 0.25)
-			(net 24 "/LDO_1.8V")
-			(pinfunction "OUT")
-			(pintype "power_out")
-			(thermal_bridge_angle 45)
-		)
-	)
 	(footprint "Connector_Molex:Molex_Nano-Fit_105309-xx04_1x04_P2.50mm_Vertical"
 		(layer "F.Cu")
@@
 		(descr "THT pad as test Point, diameter 2.0mm, hole diameter 1.0mm")
 		(tags "test point THT pad")
-		(property "Reference" "1.8V"
+		(property "Reference" "TP3"
 			(at 0 -1.998 0)
 			(layer "F.SilkS")
@@
 		(descr "THT pad as test Point, diameter 2.0mm, hole diameter 1.0mm")
 		(tags "test point THT pad")
-		(property "Reference" "IMU_SCL"
+		(property "Reference" "TP10"
 			(at 1.75 0 0)
 			(layer "F.SilkS")
@@
 		(descr "THT pad as test Point, diameter 2.0mm, hole diameter 1.0mm")
 		(tags "test point THT pad")
-		(property "Reference" "IMU_SCL"
+		(property "Reference" "TP11"
 			(at 1.75 0 0)
 			(layer "F.SilkS")
@@
 		)
 	)
+	(gr_text "+"
+		(at 178.5 105.75 0)
+		(layer "F.SilkS")
+		(effects
+			(font
+				(size 0.8 0.8)
+				(thickness 0.2)
+				(bold yes)
+			)
+			(justify left bottom mirror)
+		)
+	)
 	(gr_text "MG_CLK"
 		(at 154.75 68 90)
@@
 		)
 	)
+	(gr_text "+"
+		(at 172.75 105.75 0)
+		(layer "F.SilkS")
+		(effects
+			(font
+				(size 0.8 0.8)
+				(thickness 0.2)
+				(bold yes)
+			)
+			(justify left bottom mirror)
+		)
+	)
 	(segment
 		(start 158.95 71.55)
@@
 		(width 0.5)
 		(layer "F.Cu")
-		(net 22)
-	)
-	(segment
-		(start 170.675 83.625)
-		(end 170.75 83.7)
-		(width 0.5)
-		(layer "F.Cu")
