File: IMU_WheelSpeed/IMU_WheelSpeed.kicad_pcb (KiCad board)
At the start: 2 copper layers, 56.8 x 50 mm, 23 parts, among them J1 Conn_01x04_Socket, J2 CAN_IN, J3 Conn_01x03_Socket, J4 CAN_OUT, J5 PWR_IN, J6 PWR_OUT, J7 Conn_01x06_Socket, U1 PeripheralSOM, U4 TPS71518__SC70

Commit message: INT and moved TPs
Parts:
- removed 3.3V: VDD_3.3V, TestPoint:TestPoint_THTPad_D2.0mm_Drill1.0mm
- removed J1: Conn_01x04_Socket, Connector_Molex:Molex_Nano-Fit_105309-xx04_1x04_P2.50mm_Vertical
- added J8: IMU_CONN, Connector_Molex:Molex_Nano-Fit_105309-xx05_1x05_P2.50mm_Vertical, F.Cu at (177.2, 87.5)
- moved TP8 53.1 mm to (181.2, 105.5), turned to 0 degrees
- moved TP9 48.2 mm to (181.2, 102.0), turned to 0 degrees
- moved TP7 43.3 mm to (181.2, 98.5), turned to 0 degrees
- moved TP6 38.4 mm to (181.2, 95.0), turned to 0 degrees
- moved TP10 3.26 mm to (181.2, 91.2)
- moved TP11 3.01 mm to (181.2, 87.5)
- moved TP3 0.50 mm to (181.2, 77.5)
Connections:
- U1 pad 18: unconnected-(U1-PA2(ADC)-Pad18) -> /IMU_INT
Routing:
- net /VDD_3.3V: track 81.8 -> 51.5 mm, vias 1 -> 0
- net /MAG_CS: track 43.5 -> 65.7 mm, vias 1 -> 0
- net /MAG_CLK: track 43.8 -> 62.8 mm, vias 1 -> 0
- net /IMU_INT: track 0.00 -> 15.7 mm
- net /MAGSLV_Output: track 49.6 -> 65.2 mm, vias 1 -> 0
- net /MAGSLV_Input: track 55.8 -> 71.1 mm, vias 1 -> 0
- net GND: track 11.3 -> 5.34 mm, vias 4 -> 7
- net /IMU_I2C_SCL: track 29.0 -> 30.8 mm
- net /LDO_1.8V: track 18.4 -> 19.8 mm
- net /IMU_I2C_SDA: track 28.7 -> 29.9 mm
Other:
- board text added: "-"
- board text added: "MAGSLV_I"
- board text added: "MAGSLV_O"
- board text added: "MAG_CLK"
- board text added: "MAG_CS"
- board text removed: "MG_CLK"
- board text removed: "MG_CS"
- board text removed: "MG_SLV_IN"
- board text removed: "MG_SLV_OUT"

Commit message: fixed review stuffs
Parts:
- removed C2: 0u47, Capacitor_SMD:C_0805_2012Metric
- removed C3: 0u1, Capacitor_SMD:C_0805_2012Metric
- removed J4: CAN_OUT, UTSVT_Connectors:CONN_SD-43650-006_02_MOL
- removed J5: PWR_IN, UTSVT_Connectors:CONN_SD-43650-006_02_MOL
- removed J6: PWR_OUT, UTSVT_Connectors:CONN_SD-43650-006_02_MOL
- removed R3: 10k, Resistor_SMD:R_0805_2012Metric
- removed TP3: LDO1.8V, TestPoint:TestPoint_THTPad_D2.0mm_Drill1.0mm
- removed U4: TPS71518__SC70, UTSVT_Power:LDO_3.3_to_1.8_2.2mmx1.3mm
- added J9: CAN+POWER_OUT, UTSVT_Connectors:Molex_MicroFit3.0_1x4xP3.00mm_PolarizingPeg_Vertical, F.Cu at (169.8, 99.2)
- added R4: 10k, Resistor_SMD:R_0805_2012Metric, F.Cu at (171.2, 82.0)
- added R5: 10k, Resistor_SMD:R_0805_2012Metric, F.Cu at (168.8, 82.0)
- added TP2: VDD_3.3V, TestPoint:TestPoint_THTPad_D2.0mm_Drill1.0mm, F.Cu at (181.2, 77.5)
- J2: value CAN_IN -> Conn_01x05_Socket; footprint UTSVT_Connectors:CONN_SD-43650-006_02_MOL -> Connector_Molex:Molex_Nano-Fit_105309-xx05_1x05_P2.50mm_Vertical
- J8: value IMU_CONN -> CAN+POWER_IN; footprint Connector_Molex:Molex_Nano-Fit_105309-xx05_1x05_P2.50mm_Vertical -> UTSVT_Connectors:Molex_MicroFit3.0_1x4xP3.00mm_PolarizingPeg_Vertical
- TP10: value IMU_I2C_SDA -> I2C_SDA
- TP11: value IMU_CLK -> I2C_SCL
- moved J2 20.8 mm to (177.4, 87.5), turned to 180 degrees
- moved J8 11.8 mm to (176.2, 99.2), turned to -90 degrees
- moved R2 1.95 mm to (170.5, 85.2), turned to 180 degrees
- moved J3 0.75 mm to (176.5, 65.0)
Connections:
- J2 pad 1: /CAN_P -> GND
- J2 pad 2: /CAN_N -> Net-(J2-Pin_2)
- J3 pad 3: /VDD_3.3V -> +3.3V
- J7 pad 1: /VDD_3.3V -> +3.3V
- J8 pad 1: GND -> +12V
- J8 pad 2: /IMU_INT -> GNDPWR
- J8 pad 3: /IMU_I2C_SDA -> /CAN_P
- J8 pad 4: /IMU_I2C_SCL -> /CAN_N
- R1 pad 2: /VDD_3.3V -> +3.3V
- R2 pad 1: /IMU_I2C_SDA -> Net-(J2-Pin_2)
- R2 pad 2: /LDO_1.8V -> /IMU_INT
- U1 pad 11: unconnected-(U1-GND-Pad11) -> GND
- U1 pad 2: /VDD_3.3V -> +3.3V
- U1 pad 24: unconnected-(U1-GNDPWR-Pad24) -> GNDPWR
- U1 pad 9: /VDD_3.3V -> +3.3V
Routing:
- net +3.3V: track 0.00 -> 59.0 mm
- net /VDD_3.3V: track 51.5 -> 0.00 mm
- net GNDPWR: track 0.00 -> 19.8 mm
- net /LDO_1.8V: track 19.8 -> 0.00 mm
- net Net-(J2-Pin_2): track 0.00 -> 14.4 mm
- net /IMU_INT: track 15.7 -> 7.45 mm
- net +12V: track 13.0 -> 17.9 mm
- net /IMU_I2C_SDA: track 29.9 -> 34.4 mm
- net GND: track 5.34 -> 1.51 mm, vias 7 -> 6
- net /IMU_I2C_SCL: track 30.8 -> 31.8 mm
- net /CAN_N: track 35.8 -> 36.5 mm
- net /CAN_P: track 35.7 -> 36.4 mm
- net /LTE_D1: track 2.82 -> 2.26 mm
Other:
- board size 56.8 x 50 mm -> 57.5 x 50 mm
- board text added: "3.3V"
- board text removed: "12V_OUT"

Commit message: connectors cool I think
Routing:
- net /MAG_CS: track 65.7 -> 67.7 mm
- net /MAG_CLK: track 62.8 -> 64.8 mm
- net /MAGSLV_Output: track 65.2 -> 67.1 mm
- net /MAGSLV_Input: track 71.1 -> 72.9 mm

Commit message: just saving
Other:
- board text added: "IMU_SCL"
- board text added: "IMU_SDA"
Changed lines of the file:
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@@
 		(tags "resistor")
 		(property "Reference" "R4"
-			(at 2.5 0 180)
+			(at 2 0 180)
 			(layer "F.SilkS")
 			(effects
 				(font
-					(size 1 1)
+					(size 0.8 0.8)
 					(thickness 0.15)
 				)
@@
 		(tags "resistor")
 		(property "Reference" "R5"
-			(at -2.5 0 180)
+			(at -2 0 180)
 			(layer "F.SilkS")
 			(effects
 				(font
-					(size 1 1)
+					(size 0.8 0.8)
 					(thickness 0.15)
 				)
@@
 		(tags "resistor")
 		(property "Reference" "R2"
-			(at 0 -1.65 0)
+			(at -2.48 0 0)
 			(layer "F.SilkS")
 			(effects
 				(font
-					(size 1 1)
+					(size 0.8 0.8)
 					(thickness 0.15)
 				)
@@
 		(at 176.25 99.25 -90)
 		(property "Reference" "J8"
-			(at 12.5 -4 90)
+			(at 11.5 -0.25 90)
 			(layer "F.SilkS")
 			(effects
@@
 		(at 169.75 99.25 -90)
 		(property "Reference" "J9"
-			(at 9.5 -3.25 90)
+			(at 11.75 0 90)
 			(layer "F.SilkS")
 			(effects
@@
 			(at 1.75 0 0)
 			(layer "F.SilkS")
+			(hide yes)
 			(effects
 				(font
@@
 			(at 1.75 0 0)
 			(layer "F.SilkS")
+			(hide yes)
 			(effects
 				(font
@@
 		)
 	)
+	(gr_text "IMU_SDA"
+		(at 181.25 93 0)
+		(layer "F.SilkS")
+		(effects
+			(font
+				(size 0.5 0.5)
+				(thickness 0.125)
+			)
+		)
+	)
 	(gr_text "3.3V"
 		(at 181.25 75.75 0)
@@
 		(layer "F.SilkS")
 		(effects
+			(font
+				(size 0.5 0.5)
+				(thickness 0.125)
+			)
+		)
+	)
+	(gr_text "IMU_SCL"
+		(at 181.25 89.25 0)
+		(layer "F.SilkS")
+		(effects

Commit message: made BOM
Other:
- board text added: "."
Changed lines of the file:
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@@
+		)
+	)
+	(gr_text "."
+		(at 176 66.75 0)
+		(layer "F.SilkS")
+		(effects
+			(font
+				(size 1.5 1.5)
+				(thickness 0.3)
+				(bold yes)
+			)
+			(justify left bottom)
 		)
 	)
@@
 				(thickness 0.125)
 			)
+		)
+	)
+	(gr_text "."
+		(at 178.5 87.75 0)
+		(layer "F.SilkS")
+		(effects
+			(font
+				(size 1.5 1.5)
+				(thickness 0.3)
+				(bold yes)
+			)
+			(justify left bottom)
 		)
 	)
@@
 			)
 			(justify left bottom mirror)
+		)
+	)
+	(gr_text "."
+		(at 171 77.75 0)
+		(layer "F.SilkS")
+		(effects
+			(font
+				(size 1.5 1.5)
+				(thickness 0.3)
+				(bold yes)
+			)
+			(justify left bottom)
 		)
 	)
@@
 		)
 	)
+	(gr_text "."
+		(at 176.25 99.25 0)
+		(layer "F.SilkS")
+		(effects
+			(font
+				(size 1.5 1.5)
+				(thickness 0.3)
+				(bold yes)
+			)
+			(justify left bottom)
+		)
+	)
