File: IMU_WheelSpeed/IMU_WheelSpeed.kicad_sch (KiCad schematic)
At the start: 23 parts, among them J1 Conn_01x04_Socket, J2 CAN_IN, J3 Conn_01x03_Socket, J4 CAN_OUT, J5 PWR_IN, J6 PWR_OUT, J7 Conn_01x06_Socket, U1 PeripheralSOM, U4 TPS71518__SC70

Commit message: fixed review stuffs
Parts:
- removed C2: 0u47, Capacitor_SMD:C_0805_2012Metric, symbol Device:C
- removed C3: 0u1, Capacitor_SMD:C_0805_2012Metric, symbol Device:C
- removed J1: Conn_01x04_Socket, Connector_Molex:Molex_Nano-Fit_105309-xx04_1x04_P2.50mm_Vertical, symbol Connector:Conn_01x04_Socket
- removed J2: CAN_IN, UTSVT_Connectors:CONN_SD-43650-006_02_MOL, symbol Connector:Conn_01x02_Pin
- removed J4: CAN_OUT, UTSVT_Connectors:CONN_SD-43650-006_02_MOL, symbol Connector:Conn_01x02_Pin
- removed J5: PWR_IN, UTSVT_Connectors:CONN_SD-43650-006_02_MOL, symbol Connector:Conn_01x02_Pin
- removed J6: PWR_OUT, UTSVT_Connectors:CONN_SD-43650-006_02_MOL, symbol Connector:Conn_01x02_Pin
- removed R3: 10k, Resistor_SMD:R_0805_2012Metric, symbol Device:R
- removed TP3: LDO1.8V, TestPoint:TestPoint_THTPad_D2.0mm_Drill1.0mm, symbol Connector:TestPoint
- removed U4: TPS71518__SC70, UTSVT_Power:LDO_3.3_to_1.8_2.2mmx1.3mm, symbol Regulator_Linear:TPS71518__SC70
- added J2: Conn_01x05_Socket, Connector_Molex:Molex_Nano-Fit_105309-xx05_1x05_P2.50mm_Vertical, symbol Connector:Conn_01x05_Socket
- added J8: CAN+POWER_IN, UTSVT_Connectors:Molex_MicroFit3.0_1x4xP3.00mm_PolarizingPeg_Vertical, symbol Connector:Conn_01x04_Socket
- added J9: CAN+POWER_OUT, UTSVT_Connectors:Molex_MicroFit3.0_1x4xP3.00mm_PolarizingPeg_Vertical, symbol Connector:Conn_01x04_Socket
- added R4, R5: 10k, Resistor_SMD:R_0805_2012Metric, symbol Device:R
- TP10: value IMU_I2C_SDA -> I2C_SDA
- TP11: value IMU_CLK -> I2C_SCL
Connections:
- net LDO_1.8V is gone; now on net IMU_INT: R2.2
- net +12V: now also J8.1 (Pin_1), J9.1 (Pin_1)
- net CAN_N: now also J8.4 (Pin_4), J9.4 (Pin_4)
- net CAN_P: now also J8.3 (Pin_3), J9.3 (Pin_3)
- net GND: now also U1.11 (GND), J2.1 (Pin_1)
- net IMU_I2C_SCL: now also J2.4 (Pin_4), R4.2
- net IMU_I2C_SDA: now also J2.3 (Pin_3), R5.1; no longer R2.1
- net IMU_INT: now reaches U1.18 (PA2(ADC))
- net GNDPWR: now reaches U1.24 (GNDPWR)
- net GNDPWR: now also J8.2 (Pin_2), J9.2 (Pin_2)
- net VDD_3.3V renamed +3.3V
- net +3.3V: now also J2.5 (Pin_5), R4.1, R5.2
- new net: J2.2 (Pin_2), R2.1
- no-connect marks 11 -> 8
Other:
- note added: "CAN + POWER IN"
- note added: "CAN + POWER OUT"
- note removed: "12V Dirty"
- note removed: "12V Out"
- note removed: "3.3V to 1.8V LDO"
- note removed: "CAN Inputs"
