File: IMU_Breakout/IMU_Breakout.kicad_pcb (KiCad board)
At the start: 2 copper layers, 14.5 x 11.8 mm, 4 parts, among them J1 Conn_01x05_Socket, U1 LSM6DSL

Commit message: added through holes
Other:
- board size 14.5 x 11.8 mm -> 15.2 x 11.8 mm
Changed lines of the file:
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@@
 		)
+	)
+	(gr_circle
+		(center 141.25 91)
+		(end 141.85 91)
+		(stroke
+			(width 0.2)
+			(type solid)
+		)
+		(fill solid)
+		(layer "Edge.Cuts")
+	)
+	(gr_circle
+		(center 153.5 91)
+		(end 154.1 91)
+		(stroke
+			(width 0.2)
+			(type solid)
+		)
+		(fill solid)
+		(layer "Edge.Cuts")
 	)
 	(gr_rect
 		(start 139.75 84.5)
-		(end 154.25 96.25)
+		(end 155 96.25)
 		(stroke
 			(width 0.05)
@@
 		(layer "Edge.Cuts")
 	)
-	(gr_text "IMU\nCONN"
-		(at 152.6 90 0)
+	(gr_text "IMU CONN"
+		(at 152.25 89.25 0)
 		(layer "F.SilkS")
 		(effects
 			(font
-				(size 0.8 0.8)
+				(size 0.6 0.6)
 				(thickness 0.15)
 				(bold yes)
@@
 	)
 	(via
-		(at 152.75 91.5)
+		(at 153.5 93.5)
 		(size 0.6)
 		(drill 0.3)
